Commit message: material fixedgazebo material fix

File: giraffe_ws/src/giraffe_description/urdf/giraffe.urdf.xacro (robot description, xacro)
@@ -17,4 +17,5 @@
         </inertial>
         <visual name="shoulder_pan_shaft_visual">
+            <material name="white"/>
             <origin xyz="0.008106267583602906 7.002947095541501e-05 -0.02063014414641271" rpy="-0.002445313989558981 -0.002441606509518308 1.5715549810166236" />
             <geometry>
@@ -36,4 +37,5 @@
         </inertial>
         <visual name="wrist_2-v9_visual">
+            <material name="white"/>
             <origin xyz="0.023414439458437214 0.020117330367280157 -0.22047336491261565" rpy="1.572487094217567 -0.002449415475925335 -1.5732319621207191" />
             <geometry>
@@ -55,4 +57,5 @@
         </inertial>
         <visual name="shoulder_pan_visual">
+            <material name="white"/>
             <origin xyz="0.008145481485789195 -0.036680050862643414 -0.00010924336912160104" rpy="0.2988167777806587 1.5682395715403312 1.8720574923944682" />
             <geometry>
@@ -74,4 +77,5 @@
         </inertial>
         <visual name="shoulder_pan_actuator_visual">
+            <material name="black"/>
             <origin xyz="-0.003476575940481408 0.010236961562351949 0.006433551777754545" rpy="-1.5683547129853628 0.002445306700740462 -0.0007526837211772323" />
             <geometry>
@@ -93,4 +97,5 @@
         </inertial>
         <visual name="servo_driver_mount_visual">
+            <material name="white"/>
             <origin xyz="-0.04572865734749307 0.01766661304182639 0.0001444354796560976" rpy="-2.8427758749736154 -1.5682395715395063 -1.8720574932325007" />
             <geometry>
@@ -112,4 +117,5 @@
         </inertial>
         <visual name="base_link_visual">
+            <material name="white"/>
             <origin xyz="0.0 0.0 0.0" rpy="0.0 0.0 0.0" />
             <geometry>
@@ -131,4 +137,5 @@
         </inertial>
         <visual name="clamp_base_visual">
+            <material name="white"/>
             <origin xyz="0.029271940259570767 -0.010428927981251225 -0.04103029366675298" rpy="-1.573241641255744 -0.0007586519603592202 0.0024434618887085777" />
             <geometry>
@@ -150,4 +157,5 @@
         </inertial>
         <visual name="retainer_visual">
+            <material name="white"/>
             <origin xyz="-0.01706466684754026 -0.00484107860305972 -0.0077905820030200745" rpy="1.5708000297742428 -0.7861538278471825 3.138134460301354" />
             <geometry>
@@ -169,4 +177,5 @@
         </inertial>
         <visual name="base_brace_right_visual">
+            <material name="white"/>
             <origin xyz="-0.010547877288095388 -0.03363960101765047 0.026853826915744783" rpy="1.5683528660750305 -1.9067927307474117e-15 1.5683528658422707" />
             <geometry>
@@ -188,4 +197,5 @@
         </inertial>
         <visual name="base_brace_left_visual">
+            <material name="white"/>
             <origin xyz="-0.01038358793482051 -0.03364840729805454 -0.026904873832930984" rpy="-1.5732397875157964 3.1590454487285652e-15 -1.5683528658422705" />
             <geometry>
@@ -207,4 +217,5 @@
         </inertial>
         <visual name="shoulder_lift_visual">
+            <material name="white"/>
             <origin xyz="0.05514712621137525 0.012819765822937246 -0.018735277569727923" rpy="0.2981333907791921 -1.568233870642598 1.2702245251151756" />
             <geometry>
@@ -226,4 +237,5 @@
         </inertial>
         <visual name="elbow_link_visual">
+            <material name="white"/>
             <origin xyz="0.07316568671895611 -0.008138839143132941 -0.008134926004255659" rpy="3.139901877061385 -0.002445307403232719 1.5732397936467268" />
             <geometry>
@@ -245,4 +257,5 @@
         </inertial>
         <visual name="wrist1_link_visual">
+            <material name="white"/>
             <origin xyz="-0.028426107484972898 1.0011529867473e-05 -0.04023761155672658" rpy="0.9658415042822108 1.5678234077130215 0.9682829038963332" />
             <geometry>
@@ -264,4 +277,5 @@
         </inertial>
         <visual name="gripper_visual">
+            <material name="white"/>
             <origin xyz="6.812238235283986e-05 -4.067834789722724e-07 -0.040249938524923756" rpy="0.0016544108337975506 0.00035764457872715496 -1.7896483526330442" />
             <geometry>
@@ -283,4 +297,5 @@
         </inertial>
         <visual name="camera_mount_visual">
+            <material name="white"/>
             <origin xyz="-0.019570406927734575 -0.24492186184193013 0.014192661773020206" rpy="0.7902875010867846 1.5673407506794743 0.7861562540959603" />
             <geometry>
@@ -302,4 +317,5 @@
         </inertial>
         <visual name="shoulder_lift_actuator_visual">
+            <material name="black"/>
             <origin xyz="0.010276372105218652 -0.006412075749740908 -0.017179756791673963" rpy="0.3010460971466039 1.5682378005558886 0.29860356306546115" />
             <geometry>
@@ -321,4 +337,5 @@
         </inertial>
         <visual name="elbow_actuator_visual">
+            <material name="black"/>
             <origin xyz="-0.003540653748802356 -0.006374078860155893 0.010252185430398146" rpy="-0.0016848014948895118 -0.0024434595464297264 -0.002445314703120043" />
             <geometry>
@@ -340,4 +357,5 @@
         </inertial>
         <visual name="wrist_1_actuator_visual">
+            <material name="black"/>
             <origin xyz="-0.003485719032433359 0.006368985168599932 0.010274148214570556" rpy="-3.1391432183315153 0.002439328896973042 0.001690776503720612" />
             <geometry>
@@ -359,4 +377,5 @@
         </inertial>
         <visual name="wrist_2_actuator_visual">
+            <material name="black"/>
             <origin xyz="-0.025587058999740897 0.007181623686373453 0.010330143826798378" rpy="3.139153317375167 0.00244942797079852 -1.5691115252754138" />
             <geometry>
@@ -378,4 +397,5 @@
         </inertial>
         <visual name="finger_actuator_visual">
+            <material name="black"/>
             <origin xyz="-0.010284847372080321 -0.003459344924301089 -0.006366104550812879" rpy="1.5749305590399427 -0.0024453105374965495 1.5683547136914318" />
             <geometry>
